File: esp32_drone/esp32_drone.kicad_sch (KiCad schematic)
At the start: 0 parts

Commit message: scimetric 1
Parts:
- added FID1, FID2, FID3: 1mm Pad 2mm Mask, Fiducial:Fiducial_1mm_Mask2mm, symbol EE_NON_BOM:Fiducial-1mmPad2mmMask
- added H1, H2, H3, H4: MountingHole_2.5mm, MountingHole:MountingHole_2.5mm, symbol EE_NON_BOM:MountingHole_-_1mm_Pad_2mm_Mask
Other:
- sheet ESP32: file untitled.kicad_sch -> ESP32.kicad_sch
- sheet ESP32 ports: added USB_DN, USB_DP; removed none
- sheet Peripharals: file untitled.kicad_sch -> Peripharals.kicad_sch
- sheet Power Managment: file untitled.kicad_sch -> Power Managment.kicad_sch
- sheet Power Managment ports: added USB_DN, USB_DP; removed none
